Commit message: mesh path

File: ros2_vision_arm_control/src/urdf/dofbot.urdf (robot description, URDF)
Before this commit: robot dofbot, 6 links, 5 joints
Links:
- link base_link: geometry collision mesh filename=package://ros2_vision_arm_control/meshes/base_link.STL; visual mesh filename=package://ros2_vision_arm_control/meshes/base_link.STL
- link link1: geometry collision mesh filename=package://ros2_vision_arm_control/meshes/link1.STL; visual mesh filename=package://ros2_vision_arm_control/meshes/link1.STL
- link link2: geometry collision mesh filename=package://ros2_vision_arm_control/meshes/link2.STL; visual mesh filename=package://ros2_vision_arm_control/meshes/link2.STL
- link link3: geometry collision mesh filename=package://ros2_vision_arm_control/meshes/link3.STL; visual mesh filename=package://ros2_vision_arm_control/meshes/link3.STL
- link link4: geometry collision mesh filename=package://ros2_vision_arm_control/meshes/link4.STL; visual mesh filename=package://ros2_vision_arm_control/meshes/link4.STL
- link link5: geometry collision mesh filename=package://ros2_vision_arm_control/meshes/link5.STL; visual mesh filename=package://ros2_vision_arm_control/meshes/link5.STL

Commit message: daily update, urdf not resolved

File: ros2_vision_arm_control/src/urdf/dofbot.urdf (robot description, URDF)
Before this commit: robot dofbot, 6 links, 5 joints
Links:
- added link link6; collision box size=0.01 0.01 0.01; visual box size=0.01 0.01 0.01
Joints:
- added joint joint6: type fixed, parent link5, child link6, origin xyz=0 -0.001 -0.09 rpy=0 -1.57 0

Commit message: urdf debug, plot and check the orientation

File: ros2_vision_arm_control/src/urdf/dofbot.urdf (robot description, URDF)
Before this commit: robot dofbot, 7 links, 6 joints
Joints:
- joint joint6: origin xyz=0 -0.001 -0.09 rpy=0 -1.57 0 -> xyz=0 -0.001 0.09 rpy=0 -1.57 0
