Commit message: daily update

File: dofbot_ros2_ws/src/ros2_vision_arm_control/urdf/dofbot.urdf (robot description, URDF)
Before this commit: robot dofbot, 7 links, 6 joints
Joints:
- joint joint1: origin xyz=0 0 0.06605 rpy=-0.010805 0 0 -> xyz=0 0 0.06605 rpy=-0.010805 0 3.14159

Commit message: nodes completed

File: dofbot_ros2_ws/src/ros2_vision_arm_control/urdf/dofbot.urdf (robot description, URDF)
Before this commit: robot dofbot, 7 links, 6 joints
Joints:
- joint joint6: origin xyz=0 -0.001 0.09 rpy=0 -1.57 0 -> xyz=0 -0.001 0.105 rpy=0 -1.57 0

Commit message: daily update

File: dofbot_ros2_ws/src/ros2_vision_arm_control/urdf/dofbot.urdf (robot description, URDF)
Before this commit: robot dofbot, 7 links, 6 joints
Joints:
- joint joint1: origin xyz=0 0 0.06605 rpy=-0.010805 0 3.14159 -> xyz=0.27 0 0.06605 rpy=-0.010805 0 3.14159
